File: hardware/Telemetria Foguete/Telemetria Foguete.kicad_sch (KiCad schematic)
At the start: 18 parts, among them J10 Conn_01x01_Pin, J3 Conn_01x01_Pin, J7 Conn_01x01_Pin, J9 Conn_01x01_Pin, M1 Motor_Servo, U1 ESP32-C3-DevKitM-1, U3 SIM28ML, U4 BMP280, U5 MPU-6050, U6 SX1276

Commit message: Update Telemetria Foguete.kicad_sch
Parts:
- removed U3: SIM28ML, RF_GPS:SIM28ML, symbol RF_GPS:SIM28ML
- removed U5: MPU-6050, Sensor_Motion:InvenSense_QFN-24_4x4mm_P0.5mm, symbol Sensor_Motion:MPU-6050
- removed U6: SX1276, Package_DFN_QFN:QFN-28-1EP_6x6mm_P0.65mm_EP4.8x4.8mm, symbol RF:SX1276
- added C4: 100nF, Capacitor_THT:C_Disc_D4.7mm_W2.5mm_P5.00mm, symbol PCM_Capacitor_AKL:C_Disc_D3.0mm_W1.6mm_P2.50mm
- added J1: Antena LoRa, Connector_Coaxial:SMA_Amphenol_901-144_Vertical, symbol Connector:Conn_Coaxial_Small
- added U2: RFM95W-868S2, symbol RF_Module:RFM95W-868S2
- added U3: M8N Module, Library m1:GPS, symbol My_Library:GPS
- added U6: LSM6DS3, Package_LGA:LGA-14_3x2.5mm_P0.5mm_LayoutBorder3x4y, symbol Sensor_Motion:LSM6DS3
- U4: value BMP280 -> BMP585
- renumbered U1 to U7, U2 to U8
Connections:
- net GND: now also C4.1, U2.10 (GND), U3.1 (GND), U6.6 (GND), U6.7 (GND)
- net at U1.11 (IO10): now also U2.5 (NSS)
- net at U1.17 (IO19), U4.4 (SCK): now also U6.13 (SCL)
- net at U1.18 (IO18), U4.3 (SDI): now also U6.14 (SDA)
- net at BZ1.1 (+), U1.2 (3V3), U1.3 (3V3)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: now also C4.2, U2.13 (3.3V), U3.4 (VCC), U6.8 (VDD)
- net at U1.20 (IO4): now also U2.14 (DIO0)
- net at U1.21 (IO5): now also U2.15 (DIO1)
- net at U1.22 (IO6): now also U2.4 (SCK)
- net at U1.23 (IO7): now also U2.3 (MOSI)
- net at U1.28 (RX): now also U3.2 (TX)
- net at U1.29 (TX): now also U3.3 (RX)
- net at U1.4 (IO2): now also U2.2 (MISO)
- net at U1.5 (IO3): now also U2.6 (RESET)
- new net: J1.1 (In), U2.8 (GND)
- new net: J1.2 (Ext), U2.9 (ANT)
